File: electronics/user_interface/user_interface.kicad_pcb (KiCad board)
At the start: 2 copper layers, 80 x 80 mm, 91 parts, among them J1 Conn_01x06, J2 Conn_02x05_Odd_Even, SW1 ALPS_EC11E18244A5, U1 PCF8574, U2 PCF8574

Commit message: routing done
Routing:
- net /VDD: track 376.7 -> 402.0 mm, vias 4 -> 6
- net /!INT: track 44.5 -> 50.3 mm, vias 2 -> 3
- net /VSS: track 77.1 -> 81.9 mm
- net /VDD_RAW: track 2.92 -> 7.72 mm
- net /SDA_RAW: track 3.14 -> 7.84 mm
- net /SCL_RAW: track 2.92 -> 7.62 mm
- net /!INT_RAW: track 2.76 -> 7.46 mm
- net /SDA: track 41.9 -> 45.5 mm, vias 2 -> 3
- net /SCL: track 38.5 -> 41.9 mm, vias 2 -> 3
Changed lines of the file:
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@@
     (thickness 1.6)
     (drawings 18)
-    (tracks 540)
+    (tracks 569)
     (zones 0)
     (modules 91)
@@
   )
   (setup
-    (last_trace_width 0.127)
+    (last_trace_width 0.6)
     (user_trace_width 0.15)
     (user_trace_width 0.2)
@@
   (segment (start 173.1 93.5) (end 173.1 92.5) (width 0.6) (layer B.Cu) (net 1))
   (segment (start 172.805 93.795) (end 173.1 93.5) (width 0.6) (layer B.Cu) (net 1))
+  (segment (start 123.8 89.5) (end 119 89.5) (width 0.4) (layer B.Cu) (net 1))
   (segment (start 128.2 71.25) (end 130.7 71.25) (width 0.4) (layer B.Cu) (net 2))
   (segment (start 130.7 71.25) (end 133.3 71.25) (width 0.4) (layer B.Cu) (net 2))
@@
   (segment (start 170.4 138.7) (end 170.6 138.7) (width 0.6) (layer B.Cu) (net 2))
   (segment (start 119.5 145.3) (end 121.9 147.7) (width 0.6) (layer B.Cu) (net 2))
-  (segment (start 124.4 105.6) (end 119.5 110.5) (width 0.6) (layer B.Cu) (net 2))
   (segment (start 159.8 138.7) (end 170.6 138.7) (width 0.6) (layer B.Cu) (net 2))
   (segment (start 159.8 140) (end 159.8 138.7) (width 0.6) (layer B.Cu) (net 2))
@@
   (segment (start 119.5 143.2) (end 119.5 145.3) (width 0.6) (layer B.Cu) (net 2))
   (segment (start 119.6 123.2) (end 119.5 123.1) (width 0.6) (layer B.Cu) (net 2))
-  (segment (start 119.5 110.5) (end 119.5 123.1) (width 0.6) (layer B.Cu) (net 2))
   (segment (start 122.35 123.2) (end 119.6 123.2) (width 0.6) (layer B.Cu) (net 2))
   (segment (start 119.5 123.1) (end 119.5 143.2) (width 0.6) (layer B.Cu) (net 2))
   (segment (start 122.2 92.6) (end 122.9 93.3) (width 0.6) (layer F.Cu) (net 2))
   (segment (start 121.75 80.45) (end 122.2 80.9) (width 0.6) (layer F.Cu) (net 2))
-  (segment (start 122.2 80.9) (end 122.2 92.6) (width 0.6) (layer F.Cu) (net 2))
   (segment (start 119.625 78.325) (end 121.75 80.45) (width 0.6) (layer F.Cu) (net 2))
   (via (at 119.625 78.325) (size 0.6) (drill 0.3) (layers F.Cu B.Cu) (net 2))
@@
   (segment (start 119.625 78.325) (end 119.625 76.875) (width 0.6) (layer B.Cu) (net 2))
   (segment (start 119.625 76.875) (end 120.25 76.25) (width 0.6) (layer B.Cu) (net 2))
-  (segment (start 128.8 89.8) (end 141.5 89.8) (width 0.6) (layer F.Cu) (net 2))
   (segment (start 162 84.805) (end 157.395 84.805) (width 0.4) (layer B.Cu) (net 2))
   (segment (start 157.05 85.15) (end 157.05 85.9) (width 0.4) (layer B.Cu) (net 2))
@@
   (segment (start 170.6 138.7) (end 176.9 138.7) (width 0.6) (layer B.Cu) (net 2))
   (segment (start 176.9 138.7) (end 183.3 138.7) (width 0.6) (layer B.Cu) (net 2))
+  (via (at 122.2 82) (size 0.65) (drill 0.4) (layers F.Cu B.Cu) (net 2))
+  (segment (start 123.7 82) (end 122.2 82) (width 0.4) (layer B.Cu) (net 2))
+  (segment (start 122.2 80.9) (end 122.2 82) (width 0.6) (layer F.Cu) (net 2))
+  (segment (start 122.2 82) (end 122.2 92.6) (width 0.6) (layer F.Cu) (net 2))
+  (segment (start 119.5 110.5) (end 119.5 123.1) (width 0.6) (layer B.Cu) (net 2))
+  (segment (start 125.3 104.7) (end 119.5 110.5) (width 0.6) (layer B.Cu) (net 2))
+  (via (at 125.3 93.3) (size 0.75) (drill 0.6) (layers F.Cu B.Cu) (net 2))
+  (segment (start 122.9 93.3) (end 125.3 93.3) (width 0.6) (layer F.Cu) (net 2))
+  (segment (start 125.3 91.5) (end 125.3 93.3) (width 0.6) (layer B.Cu) (net 2))
+  (segment (start 125.3 93.3) (end 125.3 104.7) (width 0.6) (layer B.Cu) (net 2))
+  (segment (start 125.3 91.5) (end 125.3 89.5) (width 0.6) (layer B.Cu) (net 2))
+  (segment (start 141.5 89.8) (end 130.15 89.8) (width 0.6) (layer F.Cu) (net 2))
+  (segment (start 126.65 93.3) (end 125.3 93.3) (width 0.6) (layer F.Cu) (net 2))
+  (segment (start 130.15 89.8) (end 126.65 93.3) (width 0.6) (layer F.Cu) (net 2))
   (segment (start 116.27 91.04) (end 117.24 91.04) (width 0.6) (layer B.Cu) (net 3))
   (segment (start 117.7 91.5) (end 119 91.5) (width 0.6) (layer B.Cu) (net 3))
   (segment (start 117.24 91.04) (end 117.7 91.5) (width 0.6) (layer B.Cu) (net 3))
+  (segment (start 123.8 91.5) (end 119 91.5) (width 0.4) (layer B.Cu) (net 3))
   (via (at 142.8 87.6) (size 0.6) (drill 0.3) (layers F.Cu B.Cu) (net 4))
   (segment (start 131.9 87.6) (end 129.1 84.8) (width 0.4) (layer F.Cu) (net 4))
@@
   (segment (start 160.035 88.665) (end 159.8 88.9) (width 0.4) (layer B.Cu) (net 4))
   (segment (start 162 88.665) (end 160.035 88.665) (width 0.4) (layer B.Cu) (net 4))
+  (via (at 128.4 84.8) (size 0.65) (drill 0.4) (layers F.Cu B.Cu) (net 4))
+  (segment (start 129.1 84.8) (end 128.4 84.8) (width 0.4) (layer F.Cu) (net 4))
+  (segment (start 128.4 84.8) (end 127.6 84.8) (width 0.4) (layer B.Cu) (net 4))
+  (segment (start 126.3 83.5) (end 125.4 83.5) (width 0.4) (layer B.Cu) (net 4))
+  (segment (start 127.6 84.8) (end 126.3 83.5) (width 0.4) (layer B.Cu) (net 4))
+  (segment (start 125.4 82) (end 125.4 83.5) (width 0.4) (layer B.Cu) (net 4))
   (segment (start 161.995 87.4) (end 162 87.395) (width 0.4) (layer B.Cu) (net 5))
   (segment (start 142.4 88.3) (end 144.975 88.3) (width 0.4) (layer B.Cu) (net 5))
@@
   (segment (start 159.805 87.395) (end 159.8 87.4) (width 0.4) (layer B.Cu) (net 5))
   (segment (start 162 87.395) (end 159.805 87.395) (width 0.4) (layer B.Cu) (net 5))
+  (via (at 127.9 85.5) (size 0.65) (drill 0.4) (layers F.Cu B.Cu) (net 5))
+  (segment (start 128.8 85.5) (end 127.9 85.5) (width 0.4) (layer F.Cu) (net 5))
+  (segment (start 127.9 85.5) (end 125.4 85.5) (width 0.4) (layer B.Cu) (net 5))
   (via (at 142.8 89) (size 0.6) (drill 0.3) (layers F.Cu B.Cu) (net 6))
   (segment (start 142.8 89) (end 131.3 89) (width 0.4) (layer F.Cu) (net 6))
@@
   (segment (start 156.5 88.1) (end 160.3 88.1) (width 0.4) (layer F.Cu) (net 6))
   (segment (start 160.7 87.7) (end 160.7 87.1) (width 0.4) (layer F.Cu) (net 6))
+  (via (at 128.4 86.2) (size 0.65) (drill 0.4) (layers F.Cu B.Cu) (net 6))
+  (segment (start 128.5 86.2) (end 128.4 86.2) (width 0.4) (layer F.Cu) (net 6))
+  (segment (start 128.4 86.2) (end 127.55 86.2) (width 0.4) (layer B.Cu) (net 6))
+  (segment (start 126.25 87.5) (end 125.4 87.5) (width 0.4) (layer B.Cu) (net 6))
+  (segment (start 127.55 86.2) (end 126.25 87.5) (width 0.4) (layer B.Cu) (net 6))
   (segment (start 116.27 93.58) (end 117.62 93.58) (width 0.4) (layer B.Cu) (net 7))
   (segment (start 117.7 93.5) (end 119 93.5) (width 0.4) (layer B.Cu) (net 7))
@@
   (segment (start 117.6 83.5) (end 119 83.5) (width 0.4) (layer B.Cu) (net 8))
   (segment (start 117.52 83.42) (end 117.6 83.5) (width 0.4) (layer B.Cu) (net 8))
+  (segment (start 123.7 83.5) (end 119 83.5) (width 0.4) (layer B.Cu) (net 8))
   (segment (start 116.27 85.96) (end 117.14 85.96) (width 0.4) (layer B.Cu) (net 9))
   (segment (start 117.6 85.5) (end 119 85.5) (width 0.4) (layer B.Cu) (net 9))
   (segment (start 117.14 85.96) (end 117.6 85.5) (width 0.4) (layer B.Cu) (net 9))
+  (segment (start 123.7 85.5) (end 119 85.5) (width 0.4) (layer B.Cu) (net 9))
   (segment (start 116.27 88.5) (end 116.8 88.5) (width 0.4) (layer B.Cu) (net 10))
   (segment (start 117.8 87.5) (end 119 87.5) (width 0.4) (layer B.Cu) (net 10))
   (segment (start 116.8 88.5) (end 117.8 87.5) (width 0.4) (layer B.Cu) (net 10))
+  (segment (start 123.7 87.5) (end 119 87.5) (width 0.4) (layer B.Cu) (net 10))
   (segment (start 136.235 90.83) (end 134.77 90.83) (width 0.4) (layer B.Cu) (net 11))
   (segment (start 134.6 91) (end 133.65 91) (width 0.4) (layer B.Cu) (net 11))
