File: electronics/UI_small_graphic/UI_small_graphic.kicad_pcb (KiCad board)
At the start: 2 copper layers, 50 x 50 mm, 45 parts, among them J1 Conn_01x06, U1 128x32, U2 128x64, U3 PCF8574, U4 PCA9554

Commit message: small changes preparing for production
Parts:
- N2: value V20220213 -> V20220217
Routing:
- net /VSS: track 39.9 -> 39.5 mm, vias 28 -> 27

Commit message: updated versionnumber
Parts:
- N2: value V20220217 -> V20220308

Commit message: generated plots
Parts:
- N2: value V20220308 -> V20220310
