File: electronics/UI_small_graphic/UI_small_graphic.kicad_sch (KiCad schematic)
At the start: 55 parts, among them J1 Conn_01x06, U1 128x32, U2 128x64, U3 PCF8574, U4 PCA9554

Commit message: placed ESD parts, silk placed
Parts:
- N2: value V20220603 -> V20220828
Connections:
- net BUTT4: now also U4.9 (IO4)
- net VSS: now also C10.2, C9.2, D4.2 (A2), D5.2 (A2)
- no-connect marks 5 -> 4
Other:
- moved on the sheet: C7, C8, U2
Changed lines of the file:
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@@
   (no_connect (at 58.42 90.17))
   (no_connect (at 58.42 87.63))
-  (no_connect (at 58.42 133.35))
   (no_connect (at 58.42 128.27))
   (wire (pts (xy 35.56 33.02) (xy 34.29 33.02))
@@
     (stroke (width 0) (type default) (color 0 0 0 0))
   )
-  (wire (pts (xy 77.47 173.99) (xy 78.74 173.99))
+  (wire (pts (xy 93.98 156.21) (xy 95.25 156.21))
     (stroke (width 0) (type default) (color 0 0 0 0))
   )
@@
     (stroke (width 0) (type default) (color 0 0 0 0))
   )
+  (wire (pts (xy 58.42 133.35) (xy 59.69 133.35))
+    (stroke (width 0) (type default) (color 0 0 0 0))
+  )
   (wire (pts (xy 43.18 130.81) (xy 41.91 130.81))
     (stroke (width 0) (type default) (color 0 0 0 0))
@@
     (stroke (width 0) (type default) (color 0 0 0 0))
   )
-  (wire (pts (xy 105.41 163.83) (xy 106.68 163.83))
+  (wire (pts (xy 96.52 179.07) (xy 97.79 179.07))
     (stroke (width 0) (type default) (color 0 0 0 0))
   )
@@
     (stroke (width 0) (type default) (color 0 0 0 0))
   )
-  (wire (pts (xy 77.47 176.53) (xy 78.74 176.53))
+  (wire (pts (xy 93.98 158.75) (xy 95.25 158.75))
     (stroke (width 0) (type default) (color 0 0 0 0))
   )
@@
     (stroke (width 0) (type default) (color 0 0 0 0))
   )
-  (wire (pts (xy 77.47 179.07) (xy 78.74 179.07))
+  (wire (pts (xy 93.98 161.29) (xy 95.25 161.29))
     (stroke (width 0) (type default) (color 0 0 0 0))
   )
@@
     (stroke (width 0) (type default) (color 0 0 0 0))
   )
-  (wire (pts (xy 105.41 158.75) (xy 106.68 158.75))
+  (wire (pts (xy 96.52 173.99) (xy 97.79 173.99))
     (stroke (width 0) (type default) (color 0 0 0 0))
   )
@@
     (stroke (width 0) (type default) (color 0 0 0 0))
   )
-  (wire (pts (xy 96.52 163.83) (xy 97.79 163.83))
+  (wire (pts (xy 87.63 179.07) (xy 88.9 179.07))
     (stroke (width 0) (type default) (color 0 0 0 0))
   )
@@
     (stroke (width 0) (type default) (color 0 0 0 0))
   )
-  (wire (pts (xy 78.74 181.61) (xy 77.47 181.61))
+  (wire (pts (xy 95.25 163.83) (xy 93.98 163.83))
     (stroke (width 0) (type default) (color 0 0 0 0))
   )
@@
     (stroke (width 0) (type default) (color 0 0 0 0))
   )
-  (wire (pts (xy 97.79 158.75) (xy 96.52 158.75))
+  (wire (pts (xy 88.9 173.99) (xy 87.63 173.99))
     (stroke (width 0) (type default) (color 0 0 0 0))
   )
@@
     (effects (font (size 1.27 1.27)) (justify left bottom))
   )
-  (label "VSS" (at 77.47 173.99 180)
+  (label "VSS" (at 93.98 156.21 180)
     (effects (font (size 1.27 1.27)) (justify right bottom))
   )
@@
     (effects (font (size 1.27 1.27)) (justify left bottom))
   )
-  (label "3.3V" (at 96.52 163.83 180)
+  (label "3.3V" (at 87.63 179.07 180)
     (effects (font (size 1.27 1.27)) (justify right bottom))
   )
@@
     (effects (font (size 1.27 1.27)) (justify right bottom))
   )
-  (label "3.3V" (at 77.47 176.53 180)
+  (label "3.3V" (at 93.98 158.75 180)
     (effects (font (size 1.27 1.27)) (justify right bottom))
   )
@@
     (effects (font (size 1.27 1.27)) (justify right bottom))
   )
-  (label "VSS" (at 106.68 163.83 0)
+  (label "VSS" (at 97.79 179.07 0)
     (effects (font (size 1.27 1.27)) (justify left bottom))
   )
@@
     (effects (font (size 1.27 1.27)) (justify right bottom))
   )
+  (label "VSS" (at 90.17 123.19 0)
+    (effects (font (size 1.27 1.27)) (justify left bottom))
+  )
   (label "BUTT1" (at 41.91 125.73 180)
     (effects (font (size 1.27 1.27)) (justify right bottom))
@@
     (effects (font (size 1.27 1.27)) (justify left bottom))
   )
-  (label "VSS" (at 106.68 158.75 0)
+  (label "VSS" (at 97.79 173.99 0)
     (effects (font (size 1.27 1.27)) (justify left bottom))
   )
@@
     (effects (font (size 1.27 1.27)) (justify left bottom))
   )
-  (label "SDA" (at 77.47 181.61 180)
+  (label "SDA" (at 93.98 163.83 180)
     (effects (font (size 1.27 1.27)) (justify right bottom))
   )
@@
     (effects (font (size 1.27 1.27)) (justify right bottom))
   )
-  (label "SCL" (at 77.47 179.07 180)
-    (effects (font (size 1.27 1.27)) (justify right bottom))
+  (label "SCL" (at 93.98 161.29 180)
+    (effects (font (size 1.27 1.27)) (justify right bottom))
+  )
+  (label "VSS" (at 90.17 110.49 0)
+    (effects (font (size 1.27 1.27)) (justify left bottom))
   )
   (label "3.3V" (at 59.69 115.57 0)
@@
     (effects (font (size 1.27 1.27)) (justify right bottom))
   )
+  (label "BUTT4" (at 59.69 133.35 0)
+    (effects (font (size 1.27 1.27)) (justify left bottom))
+  )
   (label "VSS" (at 104.14 106.68 0)
     (effects (font (size 1.27 1.27)) (justify left bottom))
@@
     (effects (font (size 1.27 1.27)) (justify right bottom))
   )
-  (label "3.3V" (at 96.52 158.75 180)
+  (label "3.3V" (at 87.63 173.99 180)
     (effects (font (size 1.27 1.27)) (justify right bottom))
   )
@@
       (effects (font (size 1.524 1.524)))
     )
-    (property "Value" "V20220603" (id 1) (at 271.78 154.94 0)
+    (property "Value" "V20220828" (id 1) (at 271.78 154.94 0)
       (effects (font (size 1.524 1.524)))
     )
@@
     (pin "2")
   )
-  (symbol (lib_id "SquantorModules:I2C_OLED") (at 85.09 177.8 0) (unit 1)
-    (in_bom yes) (on_board yes)
-    (property "Reference" "U2" (id 0) (at 83.82 170.18 0)
+  (symbol (lib_id "SquantorModules:I2C_OLED") (at 101.6 160.02 0) (unit 1)
+    (in_bom yes) (on_board yes)
+    (property "Reference" "U2" (id 0) (at 100.33 152.4 0)
       (effects (font (size 1.27 1.27)) (justify left))
     )
-    (property "Value" "128x64" (id 1) (at 81.28 185.42 0)
+    (property "Value" "128x64" (id 1) (at 97.79 167.64 0)
       (effects (font (size 1.27 1.27)) (justify left))
     )
-    (property "Footprint" "SquantorModules:OLED_132in_128x96" (id 2) (at 83.82 177.8 0)
-      (effects (font (size 1.27 1.27)) hide)
-    )
-    (property "Datasheet" "" (id 3) (at 83.82 177.8 0)
+    (property "Footprint" "SquantorModules:OLED_132in_128x96" (id 2) (at 100.33 160.02 0)
+      (effects (font (size 1.27 1.27)) hide)
+    )
+    (property "Datasheet" "" (id 3) (at 100.33 160.02 0)
       (effects (font (size 1.27 1.27)) hide)
     )
@@
     (pin "2")
   )
-  (symbol (lib_id "Device:C") (at 101.6 158.75 270) (unit 1)
-    (in_bom yes) (on_board yes)
-    (property "Reference" "C7" (id 0) (at 104.14 157.48 90))
-    (property "Value" "10u" (id 1) (at 104.14 160.02 90))
-    (property "Footprint" "SquantorRcl:C_0603" (id 2) (at 97.79 159.7152 0)
-      (effects (font (size 1.27 1.27)) hide)
-    )
-    (property "Datasheet" "~" (id 3) (at 101.6 158.75 0)
-      (effects (font (size 1.27 1.27)) hide)
-    )
-    (pin "1")
-    (pin "2")
-  )
-  (symbol (lib_id "Device:C") (at 101.6 163.83 270) (unit 1)
-    (in_bom yes) (on_board yes)
-    (property "Reference" "C8" (id 0) (at 104.14 162.56 90))
-    (property "Value" "10u" (id 1) (at 104.14 165.1 90))
-    (property "Footprint" "SquantorRcl:C_0603" (id 2) (at 97.79 164.7952 0)
-      (effects (font (size 1.27 1.27)) hide)
-    )
-    (property "Datasheet" "~" (id 3) (at 101.6 163.83 0)
+  (symbol (lib_id "Device:C") (at 92.71 173.99 270) (unit 1)
+    (in_bom yes) (on_board yes)
+    (property "Reference" "C7" (id 0) (at 95.25 172.72 90))
+    (property "Value" "10u" (id 1) (at 95.25 175.26 90))
+    (property "Footprint" "SquantorRcl:C_0603" (id 2) (at 88.9 174.9552 0)
+      (effects (font (size 1.27 1.27)) hide)
+    )
+    (property "Datasheet" "~" (id 3) (at 92.71 173.99 0)
+      (effects (font (size 1.27 1.27)) hide)
+    )
+    (pin "1")
+    (pin "2")
+  )
+  (symbol (lib_id "Device:C") (at 92.71 179.07 270) (unit 1)
+    (in_bom yes) (on_board yes)
+    (property "Reference" "C8" (id 0) (at 95.25 177.8 90))
+    (property "Value" "10u" (id 1) (at 95.25 180.34 90))
+    (property "Footprint" "SquantorRcl:C_0603" (id 2) (at 88.9 180.0352 0)
+      (effects (font (size 1.27 1.27)) hide)
+    )
+    (property "Datasheet" "~" (id 3) (at 92.71 179.07 0)
       (effects (font (size 1.27 1.27)) hide)
     )
@@
     )
     (path "/00000000-0000-0000-0000-00005a1357a5"
-      (reference "N2") (unit 1) (value "V20220603") (footprint "SquantorLabels:Label_Generic")
+      (reference "N2") (unit 1) (value "V20220828") (footprint "SquantorLabels:Label_Generic")
     )
     (path "/00000000-0000-0000-0000-000061fa2d7e"

Commit message: updated versionnumber
Parts:
- N2: value V20220828 -> V20220916
Changed lines of the file:
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@@
       (effects (font (size 1.524 1.524)))
     )
-    (property "Value" "V20220828" (id 1) (at 271.78 154.94 0)
+    (property "Value" "V20220916" (id 1) (at 271.78 154.94 0)
       (effects (font (size 1.524 1.524)))
     )
@@
     )
     (path "/00000000-0000-0000-0000-00005a1357a5"
-      (reference "N2") (unit 1) (value "V20220828") (footprint "SquantorLabels:Label_Generic")
+      (reference "N2") (unit 1) (value "V20220916") (footprint "SquantorLabels:Label_Generic")
     )
     (path "/00000000-0000-0000-0000-000061fa2d7e"

Commit message: updated to new kicad version, updated mechanical dimensions to newer nuclone hole pattern
Parts:
- N2: value V20220916 -> V20241115
